File: stm32_st7920_rotary_temp_ctrl_hw/stm32_st7920_rotary_temp_ctrl_hw.kicad_pcb (KiCad board)
At the start: 2 copper layers, 100 x 110 mm, 145 parts, among them IC1 MAX6675, J1 USB_C_Receptacle_USB2.0, J2 CONN_01X04, Q1 C1815, Q10 C1815, Q11 C1815, Q12 C1815, Q13 IRF3205, Q2 C1815, Q3 C1815, Q4 C1815, Q5 ME15N10, Q6 C1815, Q7 C1815, Q8 IRF3205, Q9 C1815, SW1 RotaryEncoder_Switch, SW2 BT_1, SW3 BT_1, U1 XL1509, U2 74HC245, U3 STM32F103C8, U4 ASM1117, U5 MAX485, Y1 8MHz, Y2 32,768KHz

Commit message: Start layout
Parts:
- removed H1, H2: ~, Lib_Hien:KF142_9P_5.08
- added U7: ~, Lib_Hien:KF142_12P_5.08, B.Cu at (176.0, 97.4)
- added U8: ~, Lib_Hien:KF142_10P_5.08, B.Cu at (104.0, 33.9)
- moved BT1 48.1 mm to (219.8, 91.4)
- moved Y2 18.0 mm to (139.0, 76.2)
- moved C15 18.0 mm to (140.9, 77.3)
- moved C16 18.0 mm to (135.4, 77.3)
- moved J1 16.4 mm to (94.4, 106.7)
- moved C8 16.0 mm to (103.0, 114.0)
- moved R6 16.0 mm to (102.9, 105.4)
- moved D3 16.0 mm to (103.3, 111.8)
- moved R4 16.0 mm to (102.9, 109.5)
- moved R5 16.0 mm to (102.9, 107.4)
- moved R7 16.0 mm to (102.9, 103.3)
- moved R8 16.0 mm to (102.9, 101.2)
- moved L3 11.9 mm to (126.7, 77.4), turned to 90 degrees
- moved R3 11.1 mm to (109.8, 92.3)
- moved C14 11.1 mm to (120.6, 77.4), turned to -90 degrees
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Routing:
- net GND: track 0.00 -> 108.3 mm, vias 0 -> 2
- net +5V: track 0.00 -> 72.3 mm
- net +3V3: track 0.00 -> 49.7 mm
- net Net-(D13-A2): track 0.00 -> 29.6 mm
- net Net-(U1-Vi): track 0.00 -> 24.6 mm
- net +24V: track 0.00 -> 24.4 mm
- net +24V Servo: track 0.00 -> 22.0 mm
- net Net-(D12-A1): track 0.00 -> 20.1 mm
- net /SPI2_CLK: track 0.00 -> 17.4 mm
- net /SPI2_MISO: track 0.00 -> 16.9 mm, vias 0 -> 2
- net /485_RX: track 0.00 -> 16.4 mm, vias 0 -> 2
- net /MAX6675_CS: track 0.00 -> 15.7 mm
- net /PWM_Heater: track 0.00 -> 15.6 mm
- net Net-(D4-K): track 0.00 -> 14.4 mm
- net Net-(U5-RO): track 0.00 -> 14.1 mm
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
Commit message: finish v1.0
Parts:
- moved R9 79.6 mm to (110.5, 75.5)
- moved R10 79.5 mm to (108.5, 75.5)
- moved BT1 52.9 mm to (168.0, 102.0)
- moved D8 15.5 mm to (170.2, 61.2), turned to 0 degrees
- moved D10 8.93 mm to (170.2, 64.9), turned to 180 degrees
- moved SW2 6.90 mm to (135.2, 109.8)
- moved SW3 6.88 mm to (135.2, 122.8)
- moved R32 6.88 mm to (124.2, 112.3)
- moved C37 6.31 mm to (124.2, 110.3)
- moved C38 6.19 mm to (124.2, 123.2)
- moved R33 6.17 mm to (124.2, 125.2)
- moved D14 5.14 mm to (110.0, 104.7), turned to -90 degrees
- moved D16 4.92 mm to (120.0, 104.7), turned to -90 degrees
- moved D15 4.77 mm to (115.0, 104.7), turned to -90 degrees
- moved D17 4.45 mm to (169.8, 32.8), turned to 180 degrees
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Connections:
- C37 pad 1: Net-(C37-Pad1) -> /BT1
- C38 pad 1: Net-(C38-Pad1) -> /BT2
- D10 pad 1: +24V -> +24V Servo
- D17 pad 1: +24V Servo -> VIN
- D8 pad 1: +24V Servo -> VIN
- F1 pad 1: +24V Servo -> VIN
- R32 pad 1: Net-(C37-Pad1) -> /BT1
- R33 pad 1: Net-(C38-Pad1) -> /BT2
- SW2 pad 2: Net-(C37-Pad1) -> /BT1
- SW3 pad 2: Net-(C38-Pad1) -> /BT2
- U2 pad 16: /LCD_MOSI -> /LCD_DATA
- U6 pad 1: /PWM_2 -> /EXTRA_2
- U6 pad 13: /ULN_EXTRA_2 -> unconnected-(U6-O6-Pad13)
- U6 pad 14: /ULN_EXTRA_1 -> /ULN_PWM_2
- U6 pad 15: unconnected-(U6-O4-Pad15) -> /DIR_Servo
- U6 pad 17: /DIR_Servo -> /ULN_EXTRA_1
- U6 pad 18: /ULN_PWM_2 -> /ULN_EXTRA_2
- U6 pad 2: /CTR_DIR -> /EXTRA_1
- U6 pad 4: unconnected-(U6-I4-Pad4) -> /CTR_DIR
- U6 pad 5: /EXTRA_1 -> /PWM_2
- U6 pad 6: /EXTRA_2 -> GND
- U7 pad 2: /ULN_EXTRA_1 -> /ULN_EXTRA_2
- U7 pad 3: /ULN_EXTRA_2 -> /ULN_EXTRA_1
- U8 pad 1: +24V Servo -> VIN
Routing:
- net GND: track 108.3 -> 682.4 mm, vias 2 -> 267
- net +3V3: track 49.7 -> 402.1 mm, vias 0 -> 5
- net +5V: track 72.3 -> 327.2 mm, vias 0 -> 3
- net VIN: track 0.00 -> 219.1 mm, vias 0 -> 9
- net +24V: track 24.4 -> 173.4 mm, vias 0 -> 9
- net /SW_Rotory: track 0.00 -> 111.9 mm, vias 0 -> 1
- net /BT2: track 0.00 -> 103.9 mm, vias 0 -> 4
- net /BUZZER: track 0.00 -> 93.9 mm
- net /ROTORY_A: track 0.00 -> 92.1 mm, vias 0 -> 2
- net /BT1: track 0.00 -> 91.3 mm, vias 0 -> 2
- net /ROTORY_B: track 0.00 -> 82.2 mm, vias 0 -> 2
- net /YELLOW: track 0.00 -> 80.8 mm, vias 0 -> 3
- net /GREEN: track 0.00 -> 78.3 mm, vias 0 -> 3
- net /RED: track 0.00 -> 66.3 mm, vias 0 -> 1
- net /EXTRA_1: track 0.00 -> 66.3 mm, vias 0 -> 2
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- added copper zone on B.Cu, net +24V
- added copper zone on F.Cu, net +24V
- added copper zone on B.Cu, net /PWM2_OUT
- added copper zone on F.Cu, net /PWM2_OUT
- added copper zone on B.Cu, net /PWM_Heater
- added copper zone on F.Cu, net /PWM_Heater
- added copper zone on B.Cu, net /PWM_Servo
- added copper zone on F.Cu, net /PWM_Servo
- added copper zone on B.Cu, net GND
- added copper zone on F.Cu, net GND
