File: stm32_st7920_rotary_temp_ctrl_hw/stm32_st7920_rotary_temp_ctrl_hw.kicad_sch (KiCad schematic)
At the start: 134 parts, among them J1 Conn_01x04, J3 USB_OTG, J4 CONN_01X04, J5 Conn_01x05, J6 Conn_01x06_Pin, Q1 C1815, Q14 ME15N10, Q2 C1815, Q3 C1815, Q4 C1815, SW1 SW_Push, SW2 SW_Push, SW3 SW_Push, SW4 SW_Push, U1 ASM1117, U10 MAX31865_TQFN, U2 MC34063, U3 MAX485, U4 STM32F103C8, U5 PC817, U6 74HC245, U7 PC817, U8 PC817, U9 PC817, Y1 8MHz, Y2 32,768KHz

Commit message: Setup pin/port stm32f103c8t6, design schematic all block
Parts:
- removed C20, C30: 1uF, Resistor_SMD:R_0805_2012Metric, symbol linktech:C0805
- removed C32, C33: 100nF, Capacitors_SMD:C_0805_HandSoldering, symbol master-node-rescue:C
- removed C34: 100nF, Resistor_SMD:R_0805_2012Metric, symbol linktech:C0805
- removed C35: 100nF, Capacitor_SMD:C_0805_2012Metric, symbol linktech:C0805
- removed C5: 47uF, Capacitors_Tantalum_SMD:CP_Tantalum_Case-C_EIA-6032-28_Reflow, symbol master-node-rescue:CP1
- removed D10, D5, D8, D9: D_Zener, nhantt-kicad-lib:SOD-80, symbol Device:D_Zener
- removed J1: Conn_01x04, Connector_JST:JST_EH_S4B-EH_1x04_P2.50mm_Horizontal, symbol Connector_Generic:Conn_01x04
- removed J5: Conn_01x05, nhantt-kicad-lib:TerminalBlock_WAGO-236_2Stift_R5mm_5pol, symbol Connector_Generic:Conn_01x05
- removed J6: Conn_01x06_Pin, symbol Connector:Conn_01x06_Pin
- removed JP1: SolderJumper_3_Bridged12, Jumper:SolderJumper-3_P2.0mm_Open_TrianglePad1.0x1.5mm, symbol Jumper:SolderJumper_3_Bridged12
- removed JP2, JP3: SolderJumper_2_Open, Jumper:SolderJumper-2_P1.3mm_Open_Pad1.0x1.5mm, symbol Jumper:SolderJumper_2_Open
- removed L3: L600R, Inductor_SMD:L_0805_2012Metric, symbol Linktech:L0805
- removed R19: 400R, Resistor_SMD:R_0805_2012Metric, symbol Linktech:R0805
- removed R39, R40, R41, R42: 1k, Resistors_SMD:R_0805_HandSoldering, symbol master-node-rescue:R
- removed U10: MAX31865_TQFN, Package_DFN_QFN:QFN-20-1EP_5x5mm_P0.65mm_EP3.35x3.35mm, symbol Linktech:MAX31865_TQFN
- removed U5, U7, U8, U9: PC817, nhantt-kicad-lib:Optocoupler_SMD, symbol Isolator:PC817
- added C20, C30: 100nF, Capacitor_SMD:C_0805_2012Metric_Pad1.18x1.45mm_HandSolder, symbol master-node-rescue:C
- added C5: 10uF, Capacitor_SMD:C_0805_2012Metric_Pad1.18x1.45mm_HandSolder, symbol master-node-rescue:C
- added D13, D16, D18: D_Zener, nhantt-kicad-lib:SOD-80, symbol Device:D_Zener
- added D15, D17, D20: FR107, nhantt-kicad-lib:D_SMA_Standard, symbol Device:D
- added IC1: MAX6675, Lib_Hien:MAX6675, symbol Lib_Hien:MAX6675
- added J1, J2: XH-4P-2.54, Lib_Hien:XH-4P-2.54mm, symbol Lib_Hien:XH-4P-2.54
- added Q10: ME15N10, nhantt-kicad-lib:TO-252-2, symbol Transistor_FET:IRF3205
- added Q5, Q7, Q9: C1815, nhantt-kicad-lib:SOT-23, symbol master-node-rescue:C1815
- added Q6, Q8: mosfet, nhantt-kicad-lib:TO-252-2, symbol Transistor_FET:IRF3205
- added R19: 10K, Resistor_SMD:R_0805_2012Metric_Pad1.20x1.40mm_HandSolder, symbol master-node-rescue:R
- added R20, R26, R35, R36, R46, R48: 2.2k, Resistors_SMD:R_0805_HandSoldering, symbol master-node-rescue:R
- added R27, R28, R43, R44, R49, R50: 10k, Resistors_SMD:R_0805_HandSoldering, symbol master-node-rescue:R
- added R29, R45, R51: 10R, Resistors_SMD:R_0805_HandSoldering, symbol master-node-rescue:R
- added SW5: RotaryEncoder_Switch, symbol Device:RotaryEncoder_Switch
- added U5: ~, symbol Lib_Hien:XH-5P-2.54
- added U7, U8: ~, symbol Lib_Hien:XH-2P-2.54
- added V1, V2, V3, V4: VIT-M3, Lib_Hien:VIT-M3, symbol Lib_Hien:VIT-M3
- C1, C10, C11, C12, C13, C14, C16, C17, C18, C21, C22, C24, C26, C27, C28, C29, C3, C31, C36, C39, C4, C6, C8, C9: footprint Capacitors_SMD:C_0805_HandSoldering -> Capacitor_SMD:C_0805_2012Metric_Pad1.18x1.45mm_HandSolder
- C19, C23, C25, C40: footprint Capacitors_SMD:C_1206_HandSoldering -> Capacitor_SMD:C_0805_2012Metric_Pad1.18x1.45mm_HandSolder
- C37: footprint Capacitor_SMD:C_0805_2012Metric_Pad1.15x1.40mm_HandSolder -> Capacitor_SMD:C_0805_2012Metric_Pad1.18x1.45mm_HandSolder
- C38: footprint Capacitor_SMD:C_1206_3216Metric_Pad1.42x1.75mm_HandSolder -> Capacitor_SMD:C_0805_2012Metric_Pad1.18x1.45mm_HandSolder
- D1: footprint nhantt-kicad-lib:D_SMA_Standard -> Diode_SMD:D_SMA
- F1: footprint nhantt-kicad-lib:Fuse_SMD1812 -> Fuse:Fuse_1812_4532Metric_Pad1.30x3.40mm_HandSolder
- J4: footprint nhantt-kicad-lib:Header-4pin-2.54 -> Connector_PinHeader_2.54mm:PinHeader_1x04_P2.54mm_Vertical
- R21, R25: value 1k -> 10K; footprint Resistors_SMD:R_0805_HandSoldering -> Resistor_SMD:R_0805_2012Metric_Pad1.20x1.40mm_HandSolder
- R33, R38: value 1k -> 4.7K; footprint Resistors_SMD:R_0805_HandSoldering -> Resistor_SMD:R_0805_2012Metric_Pad1.20x1.40mm_HandSolder
Connections:
- net Dir_Servo is gone; now on net PWM_2: U4.10 (WKUP/USART2_CTS/ADC12_IN0/TIM2_CH1_ETR/PA0)
- net OUT1 is gone; now on net PWM_Servo: D19.2 (A), Q14.2 (D)
- net SCL is gone; now on net I2C1_SDA: U4.43 (PB7/I2C1_SDA/TIM4_CH2)
- net ctrl1 is gone; now on net PWM_2: R47.1, R52.2
- net +24V: now also D15.1 (K), D17.1 (K), D20.1 (K), R27.2, R43.2, R49.2
- net +3V3: now also R21.2, R33.2, C20.1, C5.1, IC1.4 (VCC), J2.1, R19.2, R20.2, R35.2, R46.2
- net A: now also J1.1
- net B: now also J1.2
- net DIR_Servo: now also D15.2 (A), Q6.2 (D), U5.2
- net ENA_Servo: now also D17.2 (A), Q8.2 (D), U5.1
- net GND: now also C24.2, C31.2, C20.2, C30.2, C5.2, D13.2 (A), D16.2 (A), D18.2 (A), IC1.1 (GND), IC1.2 (T-), J1.3, J2.2, Q10.3 (S), Q5.2 (E), Q6.3 (S), Q7.2 (E), Q8.3 (S), Q9.2 (E), R28.1, R44.1, R50.1, SW5.C, SW5.S2, U5.4, U7.2, U8.2; no longer C24.1, C31.1
- net PWM_2: now also R46.1, R48.2; no longer U4.12 (USART2_TX/ADC12_IN2/TIM2_CH3/PA2)
- net PWM_Servo: now also U5.3
- net SPI1_CLK: now also IC1.5 (SCK)
- net SPI1_LCD_CS: now also U4.41 (PB5/I2C1_SMBA)
- net SPI1_MISO: now also IC1.7 (DO)
- net VIN: now also U7.1
- net MAX6675_CS: now reaches U4.18 (PB0/ADC12_IN8/TIM3_CH3)
- net MAX6675_CS: now also IC1.6 (/CS)
- net SW_Rotory: now reaches U4.19 (PB1/ADC12_IN9/TIM3_CH4)
- net SW_Rotory: now also C24.1, R25.1, SW5.S1
- net ROTORY_B: now reaches R21.1
- net ROTORY_B: now also C31.1, U4.12 (USART2_TX/ADC12_IN2/TIM2_CH3/PA2), SW5.B
- net I2C1_SDA: now reaches R33.1
- net I2C1_SDA: now also J2.4
- net BT1 renamed BT_LEFT
- net BT_LEFT: now also U4.27 (PB14/SPI2_MISO/USART3_RTS/TIM1_CH2N); no longer U4.25 (PB12/SPI2_NSS/I2C2_SMBA/USART3_CK/TIM1_BKIN)
- net BT2 renamed BT_RIGHT
- net BT_RIGHT: now also U4.28 (PB15/SPI2_MOSI/TIM1_CH3N); no longer U4.26 (PB13/SPI2_SCK/USART3_CTS/TIM1_CH1N)
- net BT3 renamed BT_UP
- net BT_UP: now also U4.26 (PB13/SPI2_SCK/USART3_CTS/TIM1_CH1N); no longer U4.27 (PB14/SPI2_MISO/USART3_RTS/TIM1_CH2N)
- net BT4 renamed BT_DOWN
- net BT_DOWN: now also U4.25 (PB12/SPI2_NSS/I2C2_SMBA/USART3_CK/TIM1_BKIN); no longer U4.28 (PB15/SPI2_MOSI/TIM1_CH3N)
- net Buzzer renamed BUZZER
- net PWM_1_Servo renamed ROTORY_A
- net ROTORY_A: now also C30.1, R19.1, SW5.A
- net PWM_3 renamed CTR_DIR
- net CTR_DIR: now also R35.1, R36.2
- net PWM_Ctr_Thermistor renamed PWM_1
- net SDA renamed I2C1_SCL
- net I2C1_SCL: now also R38.1, J2.3
- net SPI1_CS renamed CTR_ENA
- net CTR_ENA: now also R20.1, R26.2
- removed net input1: C24.2, R25.1
- removed net input2: C31.2, R38.1
- new net: D18.1 (K), Q9.3 (C), R49.1, R50.2, R51.1
- new net: D13.1 (K), Q5.3 (C), R27.1, R28.2, R29.1
- new net: D16.1 (K), Q7.3 (C), R43.1, R44.2, R45.1
- new net: Q8.1 (G), R45.2
- new net: Q7.1 (B), R36.1
- new net: Q10.1 (G), R51.2
- new net: Q9.1 (B), R48.1
- new net: Q5.1 (B), R26.1
- new net: Q6.1 (G), R29.2
- new net +24V Servo: U5.5
- new net PWM_Heater: D20.2 (A), Q10.2 (D), U8.1
- new net T+: IC1.3 (T+), J1.4
- no-connect marks 11 -> 9
Other:
- note added: "Connecter"
- note added: "Control Heater"
- note added: "MAX6675"
- note added: "RS485 - Control Fan"
- note added: "Rotory encoder switch"
- note removed: "C35 = 100nF for 100 ohm RTD, 10nF for 1K"
- note removed: "JP1 to GND for 2/4-wire, to FORCE+ for 3-wire"
- note removed: "JP2 to closed on 2-wire"
- note removed: "JP3 to closed on 2/3-wire setup, open for 4-wire"
- note removed: "PT100/PT1000"
- note removed: "R3 = 4 x resistance at 0*C (so 400R for a 100 Ohm RTD). Use high quality 1% or better resistor"
- note removed: "RS485"
- moved on the sheet: D14, D19, D6, J4, Q1, Q14, R30, R47, R52, R59, R60, R66

Commit message: Delete block buton, Modify block connecter, Modify Block Power input, Update ALL footprint
Parts:
- removed C14, C29, C3, C37, C9: 100nF, Capacitor_SMD:C_0805_2012Metric_Pad1.18x1.45mm_HandSolder, symbol master-node-rescue:C
- removed C7: 100uF, nhantt-kicad-lib:CP_Elec_8x10, symbol master-node-rescue:CP1
- removed C8: 33p, Capacitor_SMD:C_0805_2012Metric_Pad1.18x1.45mm_HandSolder, symbol master-node-rescue:C
- removed D13, D16: D_Zener, nhantt-kicad-lib:SOD-80, symbol Device:D_Zener
- removed D15, D17: FR107, nhantt-kicad-lib:D_SMA_Standard, symbol Device:D
- removed D3: 1N5819/SS14, nhantt-kicad-lib:D_SMB_Handsoldering, symbol master-node-rescue:D_Schottky
- removed D4: D_ALT, nhantt-kicad-lib:SOD-80, symbol master-node-rescue:D_ALT
- removed J1, J2: XH-4P-2.54, Lib_Hien:XH-4P-2.54mm, symbol Lib_Hien:XH-4P-2.54
- removed J3: USB_OTG, nhantt-kicad-lib:USB_Micro-B, symbol master-node-rescue:USB_OTG
- removed L1: L, nhantt-kicad-lib:Inductor_5.2x5.8x4.5, symbol master-node-rescue:L
- removed Q6, Q8: mosfet, nhantt-kicad-lib:TO-252-2, symbol Transistor_FET:IRF3205
- removed R1: 0.15, Resistors_SMD:R_1206_HandSoldering, symbol master-node-rescue:R
- removed R10: 1.5k, Resistors_SMD:R_0805_HandSoldering, symbol master-node-rescue:R
- removed R14, R17: 22R, Resistors_SMD:R_0805_HandSoldering, symbol master-node-rescue:R
- removed R18, R23, R24, R28, R32, R44: 10k, Resistors_SMD:R_0805_HandSoldering, symbol master-node-rescue:R
- removed R29, R45: 10R, Resistors_SMD:R_0805_HandSoldering, symbol master-node-rescue:R
- removed R3: 3k, Resistors_SMD:R_0805_HandSoldering, symbol master-node-rescue:R
- removed R4: 1k, Resistors_SMD:R_0805_HandSoldering, symbol master-node-rescue:R
- removed SW1, SW2, SW3, SW4: SW_Push, Buttons_Switches_THT:SW_PUSH-12mm_Wuerth-430476085716, symbol master-node-rescue:SW_Push
- removed U2: MC34063, nhantt-kicad-lib:SOIC-8_3.9x4.9mm_Pitch1.27mm, symbol master-node-rescue:MC34063
- removed U5: ~, symbol Lib_Hien:XH-5P-2.54
- removed U7, U8: ~, symbol Lib_Hien:XH-2P-2.54
- added C10: 180uF_35v, Capacitor_SMD:CP_Elec_6.3x9.9, symbol Device:C_Polarized_Small_US
- added C11: 100nF, Capacitor_SMD:C_0805_2012Metric_Pad1.18x1.45mm_HandSolder, symbol ph_chemical_refrigerator_relay_hw-rescue:C0805-ph_kicad_lib
- added C5: 1uF_50V, Capacitor_SMD:C_0805_2012Metric_Pad1.18x1.45mm_HandSolder, symbol Device:C_Small
- added C6: 220uF_50V, Capacitor_SMD:CP_Elec_8x10.5, symbol Device:C_Polarized_Small_US
- added C7: 100nF, Capacitor_SMD:C_0805_2012Metric_Pad1.18x1.45mm_HandSolder, symbol Device:C_Small
- added D3: 1N4007_T7, Diode_SMD:D_SOD-123F, symbol Device:D
- added D4: 1N5820, Diode_SMD:D_SMA, symbol Diode:1N5820
- added H1, H2: ~, Lib_Hien:KF142_9P_5.08, symbol Lib_Hien:KF142-5.08-9P
- added J1: USB_C_Receptacle_USB2.0, Connector_USB:USB_C_Receptacle_GCT_USB4105-xx-A_16P_TopMnt_Horizontal, symbol Connector:USB_C_Receptacle_USB2.0
- added L1: L_Ferrite, Inductor_THT:L_Radial_D7.5mm_P3.50mm_Fastron_07P, symbol Device:L_Ferrite
- added L2: 68uH_2A, Inductor_SMD:L_Bourns-SRU8028_8.0x8.0mm, symbol Device:L
- added R4, R5: 5.1K, Resistor_SMD:R_0805_2012Metric_Pad1.20x1.40mm_HandSolder, symbol Device:R
- added R6, R7: 22R, Resistor_SMD:R_0805_2012Metric_Pad1.20x1.40mm_HandSolder, symbol master-node-rescue:R
- added R8: 1.5k, Resistor_SMD:R_0805_2012Metric_Pad1.20x1.40mm_HandSolder, symbol master-node-rescue:R
- added U1: XL1509, Package_SO:SOIC-8-1EP_3.9x4.9mm_P1.27mm_EP2.41x3.81mm, symbol D_H_Lib_:XL1509
- BT1: value 3V3 -> CR1220; footprint nhantt-kicad-lib:BT3V3 -> Lib_Hien:CR1220
- C1: renamed from C2; footprint nhantt-kicad-lib:CP_Elec_8x10.5 -> Capacitor_SMD:CP_Elec_8x10.5
- C8: renamed from C15; footprint Capacitors_SMD:C_0805_HandSoldering -> Capacitor_SMD:C_0805_2012Metric_Pad1.18x1.45mm_HandSolder
- D1: renamed from D21; footprint nhantt-kicad-lib:D_SMA_Standard -> Diode_SMD:D_SMB
- D10: renamed from D19; footprint nhantt-kicad-lib:D_SMA_Standard -> Diode_SMD:D_SMA
- D11: renamed from D7; footprint nhantt-kicad-lib:D_SOD-323F -> Diode_SMD:D_SOD-323F
- D5: renamed from D2; footprint LEDs:LED_0805 -> LED_SMD:LED_0805_2012Metric_Pad1.15x1.40mm_HandSolder
- D6: renamed from D18; footprint nhantt-kicad-lib:SOD-80 -> Diode_SMD:D_SC-80_HandSoldering
- D7: renamed from D14; footprint nhantt-kicad-lib:SOD-80 -> Diode_SMD:D_SC-80_HandSoldering
- D8: renamed from D6; footprint LEDs:LED_0805 -> LED_SMD:LED_0805_2012Metric_Pad1.15x1.40mm_HandSolder
- D9: renamed from D20; footprint nhantt-kicad-lib:D_SMA_Standard -> Diode_SMD:D_SMA
- L3: renamed from L2; footprint Resistors_SMD:R_0805_HandSoldering -> Resistor_SMD:R_0805_2012Metric_Pad1.20x1.40mm_HandSolder
- Q1: renamed from Q3; footprint nhantt-kicad-lib:SOT-23 -> Package_TO_SOT_SMD:SOT-23
- Q2: renamed from Q9; footprint nhantt-kicad-lib:SOT-23 -> Package_TO_SOT_SMD:SOT-23
- Q3: renamed from Q1; footprint nhantt-kicad-lib:SOT-23 -> Package_TO_SOT_SMD:SOT-23
- Q4: renamed from Q10; footprint nhantt-kicad-lib:TO-252-2 -> Package_TO_SOT_SMD:TO-252-2
- Q5: renamed from Q14; footprint nhantt-kicad-lib:TO-252-2 -> Package_TO_SOT_SMD:TO-252-2
- Q6: renamed from Q2; footprint nhantt-kicad-lib:SOT-23 -> Package_TO_SOT_SMD:SOT-23
- Q7: renamed from Q4; footprint nhantt-kicad-lib:SOT-23 -> Package_TO_SOT_SMD:SOT-23
- Q8: renamed from Q7; footprint nhantt-kicad-lib:SOT-23 -> Package_TO_SOT_SMD:SOT-23
- Q9: renamed from Q5; footprint nhantt-kicad-lib:SOT-23 -> Package_TO_SOT_SMD:SOT-23
- R1: renamed from R34; footprint Resistors_SMD:R_0805_HandSoldering -> Resistor_SMD:R_0805_2012Metric_Pad1.20x1.40mm_HandSolder
- R11: renamed from R5; footprint Resistors_SMD:R_0805_HandSoldering -> Resistor_SMD:R_0805_2012Metric_Pad1.20x1.40mm_HandSolder
- R12: renamed from R6; footprint Resistors_SMD:R_0805_HandSoldering -> Resistor_SMD:R_0805_2012Metric_Pad1.20x1.40mm_HandSolder
- R16: renamed from R2; footprint Resistors_SMD:R_0805_HandSoldering -> Resistor_SMD:R_0805_2012Metric_Pad1.20x1.40mm_HandSolder
- R17: renamed from R46; footprint Resistors_SMD:R_0805_HandSoldering -> Resistor_SMD:R_0805_2012Metric_Pad1.20x1.40mm_HandSolder
- R18: renamed from R48; footprint Resistors_SMD:R_0805_HandSoldering -> Resistor_SMD:R_0805_2012Metric_Pad1.20x1.40mm_HandSolder
- R19: renamed from R52; footprint Resistors_SMD:R_0805_HandSoldering -> Resistor_SMD:R_0805_2012Metric_Pad1.20x1.40mm_HandSolder
- R2: renamed from R31; footprint Resistors_SMD:R_0805_HandSoldering -> Resistor_SMD:R_0805_2012Metric_Pad1.20x1.40mm_HandSolder
- R20: renamed from R49; footprint Resistors_SMD:R_0805_HandSoldering -> Resistor_SMD:R_0805_2012Metric_Pad1.20x1.40mm_HandSolder
- R21: renamed from R59; footprint Resistors_SMD:R_0805_HandSoldering -> Resistor_SMD:R_0805_2012Metric_Pad1.20x1.40mm_HandSolder
- R22: renamed from R30; footprint Resistors_SMD:R_0805_HandSoldering -> Resistor_SMD:R_0805_2012Metric_Pad1.20x1.40mm_HandSolder
- R23: renamed from R13; footprint Resistors_SMD:R_0805_HandSoldering -> Resistor_SMD:R_0805_2012Metric_Pad1.20x1.40mm_HandSolder
- R24: renamed from R50; footprint Resistors_SMD:R_0805_HandSoldering -> Resistor_SMD:R_0805_2012Metric_Pad1.20x1.40mm_HandSolder
- R25: renamed from R60; footprint Resistors_SMD:R_0805_HandSoldering -> Resistor_SMD:R_0805_2012Metric_Pad1.20x1.40mm_HandSolder
- R26: renamed from R51; footprint Resistors_SMD:R_0805_HandSoldering -> Resistor_SMD:R_0805_2012Metric_Pad1.20x1.40mm_HandSolder
- R27: renamed from R66; footprint Resistors_SMD:R_0805_HandSoldering -> Resistor_SMD:R_0805_2012Metric_Pad1.20x1.40mm_HandSolder
- R28: renamed from R15; footprint Resistors_SMD:R_0805_HandSoldering -> Resistor_SMD:R_0805_2012Metric_Pad1.20x1.40mm_HandSolder
- R29: renamed from R11; footprint Resistors_SMD:R_0805_HandSoldering -> Resistor_SMD:R_0805_2012Metric_Pad1.20x1.40mm_HandSolder
- R3: renamed from R37; footprint Resistors_SMD:R_0805_HandSoldering -> Resistor_SMD:R_0805_2012Metric_Pad1.20x1.40mm_HandSolder
- R30: renamed from R9; footprint Resistors_SMD:R_0805_HandSoldering -> Resistor_SMD:R_0805_2012Metric_Pad1.20x1.40mm_HandSolder
- R31: renamed from R8; footprint Resistors_SMD:R_0805_HandSoldering -> Resistor_SMD:R_0805_2012Metric_Pad1.20x1.40mm_HandSolder
- R32: renamed from R35; footprint Resistors_SMD:R_0805_HandSoldering -> Resistor_SMD:R_0805_2012Metric_Pad1.20x1.40mm_HandSolder
- R33: renamed from R20; footprint Resistors_SMD:R_0805_HandSoldering -> Resistor_SMD:R_0805_2012Metric_Pad1.20x1.40mm_HandSolder
- R34: renamed from R36; footprint Resistors_SMD:R_0805_HandSoldering -> Resistor_SMD:R_0805_2012Metric_Pad1.20x1.40mm_HandSolder
- R35: renamed from R26; footprint Resistors_SMD:R_0805_HandSoldering -> Resistor_SMD:R_0805_2012Metric_Pad1.20x1.40mm_HandSolder
- R36: renamed from R7; footprint Resistors_SMD:R_0805_HandSoldering -> Resistor_SMD:R_0805_2012Metric_Pad1.20x1.40mm_HandSolder
- R37: renamed from R12; footprint Resistors_SMD:R_0805_HandSoldering -> Resistor_SMD:R_0805_2012Metric_Pad1.20x1.40mm_HandSolder
- R38: renamed from R16; footprint Resistors_SMD:R_0805_HandSoldering -> Resistor_SMD:R_0805_2012Metric_Pad1.20x1.40mm_HandSolder
- R39: renamed from R43; footprint Resistors_SMD:R_0805_HandSoldering -> Resistor_SMD:R_0805_2012Metric_Pad1.20x1.40mm_HandSolder
- R40: renamed from R22; footprint Resistors_SMD:R_0805_HandSoldering -> Resistor_SMD:R_0805_2012Metric_Pad1.20x1.40mm_HandSolder
- R41: renamed from R27; footprint Resistors_SMD:R_0805_HandSoldering -> Resistor_SMD:R_0805_2012Metric_Pad1.20x1.40mm_HandSolder
- RV1: footprint (none) -> Potentiometer_SMD:Potentiometer_ACP_CA14-VSMD_Vertical_Hole
- Re1: renamed from R47; footprint Resistors_SMD:R_0805_HandSoldering -> Resistor_SMD:R_0805_2012Metric_Pad1.20x1.40mm_HandSolder
- ST1: renamed from ST79201; footprint nhantt-kicad-lib:ST7920 -> Lib_Hien:GLCD-ST7920
- U2: renamed from U6; footprint (none) -> Package_SO:HTSSOP-20-1EP_4.4x6.5mm_P0.65mm_EP2.74x3.86mm
- U3: renamed from U4; footprint nhantt-kicad-lib:LQFP-48_7x7mm_Pitch0.5mm -> Package_QFP:LQFP-48-1EP_7x7mm_P0.5mm_EP3.6x3.6mm_ThermalVias
- U4: renamed from U1; footprint nhantt-kicad-lib:SOT-223 -> Package_TO_SOT_SMD:SOT-223
- Y1: footprint nhantt-kicad-lib:Crystal_SMD_HC49-SD -> Crystal:Crystal_SMD_5032-2Pin_5.0x3.2mm_HandSoldering
- Y2: footprint nhantt-kicad-lib:Crystal_SMD_HC49-SD -> Crystal:Crystal_DS15_D1.5mm_L5.0mm_Horizontal
- renumbered C20 to C12, C12 to C14, C26 to C15, C27 to C16, C16 to C19, C25 to C2, C4 to C20, C5 to C22, C31 to C23, C22 to C24, C30 to C25, C23 to C26, C10 to C27, C11 to C28, C39 to C29, C28 to C3, C38 to C30, C40 to C31, C6 to C32, C24 to C33, C36 to C34, C1 to C4, C19 to C9, D11 to D13, D1 to D2, F3 to F2, F2 to F3, J4 to J2, R38 to R10, R21 to R13, R19 to R14, R25 to R15, R33 to R9, SW5 to SW1, U3 to U5
Connections:
- net +24V: now also C5.1, L1.1
- net +24V Servo: now also H2.4
- net +3V3: now also H2.7
- net +5V: now also C10.1, C11.1, D3.1 (K), L2.2, U1.3 (FB)
- net A: now also H1.3
- net B: now also H1.4
- net DIR_Servo: now also Q9.3 (C), R41.1, H2.2
- net ENA_Servo: now also Q8.3 (C), R39.1, H2.1
- net GND: now also C10.2, C11.2, C5.2, C6.2, C7.2, D4.2 (A), H1.5, H1.8, H1.9 (8), H2.5, H2.6, J1.A1 (GND), J1.A12 (GND), J1.A8 (SBU1), J1.B1 (GND), J1.B12 (GND), J1.B8 (SBU2), J1.S1 (SHIELD), R4.1, R5.1, U1.4 (On/Off), U1.5 (GND); no longer U2.7 (A5), U2.8 (A6), U2.9 (A7)
- net I2C1_SCL: now also H2.8
- net I2C1_SDA: now also H2.9 (8)
- net PWM_1: now also R17.1, R18.2
- net PWM_2: no longer R17.1, R18.2
- net PWM_Heater: now also H1.7
- net PWM_Servo: now also H2.3
- net T+: now also H1.6
- net USBDM: now also R6.1
- net USBDP: now also R7.1
- net USB_DIS: now also R8.1
- net BT_DOWN: no longer names the net of U3.25 (PB12/SPI2_NSS/I2C2_SMBA/USART3_CK/TIM1_BKIN)
- net BT_LEFT renamed BT1
- net BT_RIGHT renamed BT2
- net BT_UP: no longer names the net of U3.26 (PB13/SPI2_SCK/USART3_CTS/TIM1_CH1N)
- new net: D4.1 (K), L2.1, U1.2 (Vo)
- new net: J1.A5 (CC1), R4.2
- new net: J1.B5 (CC2), R5.2
- new net: D3.2 (A), J1.A4 (VBUS), J1.A9 (VBUS), J1.B4 (VBUS), J1.B9 (VBUS)
- new net: J1.A6 (D+), J1.B6 (D+), R7.2, R8.2
- new net: J1.A7 (D-), J1.B7 (D-), R6.2
- new net: C6.1, C7.1, L1.2, U1.1 (Vi)
- no-connect marks 9 -> 15
Other:
- note added: "UBS - Type C"
- note removed: "Button left, right, up, right"
- note removed: "UBS"
- moved on the sheet: C1, C2, C3, C4, C8, C9, D1, D10, D2, D7, F1, Q1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

Commit message: modify block control servo, block control heater, create button, create 3 led status
Parts:
- removed D8: LED, LED_SMD:LED_0805_2012Metric_Pad1.15x1.40mm_HandSolder, symbol master-node-rescue:LED
- removed D9: FR107, Diode_SMD:D_SMA, symbol Device:D
- removed Q4: ME15N10, Package_TO_SOT_SMD:TO-252-2, symbol Transistor_FET:IRF3205
- removed Q8: C1815, Package_TO_SOT_SMD:SOT-23, symbol master-node-rescue:C1815
- added C35: 220uF_50V, Capacitor_SMD:CP_Elec_8x10.5, symbol Device:C_Polarized_Small_US
- added C36: 100nF, Capacitor_SMD:C_0805_2012Metric_Pad1.18x1.45mm_HandSolder, symbol Device:C_Small
- added C37, C38: 100nF, Capacitor_SMD:C_0805_2012Metric_Pad1.18x1.45mm_HandSolder, symbol master-node-rescue:C
- added D14, D15, D16: LED, LED_THT:LED_D3.0mm, symbol master-node-rescue:LED
- added D17, D8: SS54, Diode_SMD:D_SMA, symbol Diode:1N5711
- added D9: 12V, Diode_SMD:D_SMA, symbol Device:D_Zener
- added Q10, Q11, Q12, Q4: C1815, Package_TO_SOT_SMD:SOT-23, symbol master-node-rescue:C1815
- added Q13, Q8: IRF3205, Package_TO_SOT_SMD:TO-263-2, symbol Transistor_FET:IRF3205
- added R42, R44, R45, R46: 10K, Resistor_SMD:R_0805_2012Metric_Pad1.20x1.40mm_HandSolder, symbol master-node-rescue:R
- added R43: 2.2k, Resistor_SMD:R_0805_2012Metric_Pad1.20x1.40mm_HandSolder, symbol master-node-rescue:R
- added SW2, SW3: BT_1, Lib_Hien:SW_PUSH-12.3mm, symbol Switch:SW_Push
- added U6: ~, Lib_Hien:ULN2803AD, symbol Lib_Hien:ULN2803AD
- D6: value D_Zener -> 12V; footprint Diode_SMD:D_SC-80_HandSoldering -> Diode_SMD:D_SMA
- R18, R32, R33: value 2.2k -> 10K
- R20, R41: value 10k -> 2.2k
- R22: value 1k -> 10K
- R24: value 10k -> 10K
- R26: value 10R -> 10K
- R34, R35: value 2.2k -> 1k
- R39: value 10k -> 1k
- RV1: value 100K -> 100K/EVM3E-104; footprint Potentiometer_SMD:Potentiometer_ACP_CA14-VSMD_Vertical_Hole -> Lib_Hien:TRIMMER-EVM3E-104
- SW1: footprint (none) -> Lib_Hien:Rotary-Encoder-SW
Connections:
- net +24V: now also R18.1, C35.1, C36.1, Q11.3 (C), Q4.3 (C), R42.1, U6.10 (COM); no longer R20.2, R39.2, R41.2
- net +3V3: now also R34.2, R35.2, R39.2; no longer R17.2, R22.2
- net BT1: now also U3.21 (PB10/I2C2_SCL/USART3_TX); no longer U3.27 (PB14/SPI2_MISO/USART3_RTS/TIM1_CH2N)
- net BT2: now also U3.22 (PB11/I2C2_SDA/USART3_RX); no longer U3.28 (PB15/SPI2_MOSI/TIM1_CH3N)
- net CTR_DIR: now also U6.2 (I2); no longer R32.1, R34.2
- net CTR_ENA: now also U6.3 (I3); no longer R33.1, R35.2
- net DIR_Servo: now also U6.17 (O2); no longer Q9.3 (C), R41.1
- net ENA_Servo: now also U6.16 (O3); no longer R39.1
- net GND: now also H1.2, Q9.3 (C), R26.1, C35.2, C36.2, C37.2, C38.2, D9.2 (A), Q10.2 (E), Q12.3 (C), Q13.3 (S), Q8.3 (S), R45.1, SW2.1, SW3.1, U6.9 (GND); no longer Q9.2 (E), R24.1
- net MAX6675_CS: now also U3.25 (PB12/SPI2_NSS/I2C2_SMBA/USART3_CK/TIM1_BKIN); no longer U3.18 (PB0/ADC12_IN8/TIM3_CH3)
- net PWM_1: now also U6.4 (I4); no longer R17.1, R18.2
- net PWM_2: now also U6.1 (I1); no longer R19.2, Re1.1
- net SPI1_CLK: no longer IC1.5 (SCK)
- net VIN: now also H1.1, D17.1 (K), D8.1 (K)
- net SPI2_CLK: now reaches U3.26 (PB13/SPI2_SCK/USART3_CTS/TIM1_CH1N)
- net SPI2_CLK: now also IC1.5 (SCK)
- net YELLOW: now reaches U3.45 (PB8/TIM4_CH3)
- net YELLOW: now also D16.1 (K)
- net GREEN: now reaches U3.46 (PB9/TIM4_CH4)
- net GREEN: now also D15.1 (K)
- net at R22.1: now also Q4.2 (E)
- net at R34.1: now also D14.2 (A)
- net at R26.2: now also D6.1 (K), Q9.2 (E), R22.2, R24.1
- net at Q2.1 (B): now also R17.1; no longer R18.1
- net at Q9.1 (B): now also R20.1, Q4.1 (B); no longer R35.1
- net LED_STT renamed RED
- net RED: now also D14.1 (K)
- net SPI1_MISO renamed PWM_3
- net PWM_3: no longer IC1.7 (DO)
- new net: D16.2 (A), R39.1
- new net: C37.1, R32.1, SW2.2
- new net: D9.1 (K), Q12.2 (E), R44.2, R45.2, R46.1
- new net: Q8.1 (G), R24.2
- new net: Q13.1 (G), R46.2
- new net: C38.1, R33.1, SW3.2
- new net: Q11.2 (E), R44.1
- new net: D15.2 (A), R35.1
- new net: Q2.3 (C), R18.2, R20.2
- new net: Q11.1 (B), Q12.1 (B), R43.1
- new net: Q10.3 (C), R42.2, R43.2
- new net: Q10.1 (B), R41.1
- new net EXTRA_1: U3.18 (PB0/ADC12_IN8/TIM3_CH3), U6.5 (I5)
- new net EXTRA_2: U3.28 (PB15/SPI2_MOSI/TIM1_CH3N), U6.6 (I6)
- new net PWM1: R17.2
- new net PWM1_OUT: D8.2 (A), Q8.2 (D)
- new net PWM2: R41.2
- new net PWM2_OUT: D17.2 (A), Q13.2 (D)
- new net SPI2_MISO: IC1.7 (DO), U3.27 (PB14/SPI2_MISO/USART3_RTS/TIM1_CH2N)
- new net ULN_EXTRA_1: U6.14 (O5)
- new net ULN_EXTRA_2: U6.13 (O6)
- new net ULN_EXTRA_3: U6.12 (O7)
- new net ULN_EXTRA_4: U6.11 (O8)
- new net ULN_PWM_2: R19.2, Re1.1, U6.18 (O1)
Other:
- note added: "BUTTON"
- note added: "LED STATUS"
- moved on the sheet: C20, C22, C30, C32, D10, D5, D7, H1, H2, Q3, Q5, R16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

Commit message: Xep xong linh kien ben PCB, con mot vai output chua cho ra terminal
Parts:
- removed C35: 220uF_50V, Capacitor_SMD:CP_Elec_8x10.5, symbol Device:C_Polarized_Small_US
- added C35: 10uF, Capacitor_SMD:C_0805_2012Metric_Pad1.18x1.45mm_HandSolder, symbol Device:C_Small
- D6, D9: footprint Diode_SMD:D_SMA -> Diode_SMD:D_SC-80_HandSoldering
Connections:
- net PWM1 is gone; now on net PWM_1: R17.2
- net PWM1_OUT is gone; now on net PWM_Heater: D8.2 (A), Q8.2 (D)
- net PWM2 is gone; now on net PWM_3: R41.2
- net VIN is gone; now on net +24V Servo: D17.1 (K), D8.1 (K), F1.1, H1.1
- net +24V: now also C35.1
- net GND: now also H1.6, U6.7 (I7), U6.8 (I8), C35.2; no longer H1.5, H1.9 (8)
- net PWM2_OUT: now also H1.9 (8)
- net PWM_1: no longer U6.4 (I4)
- net T+: now also H1.5; no longer H1.6
- net ULN_EXTRA_3: no longer names the net of U6.12 (O7)
- net ULN_EXTRA_4: no longer names the net of U6.11 (O8)
- no-connect marks 15 -> 17
Other:
- moved on the sheet: D11, LS1, Q7, R40

Commit message: Start layout
Parts:
- removed H1, H2: ~, Lib_Hien:KF142_9P_5.08, symbol Lib_Hien:KF142-5.08-9P
- added U7: ~, Lib_Hien:KF142_12P_5.08, symbol Lib_Hien:XH-12P-2.54
- added U8: ~, Lib_Hien:KF142_10P_5.08, symbol Lib_Hien:XH-10P-2.54
Connections:
- net +24V Servo: now also U7.7, U8.1
- net +3V3: now also U8.8
- net A: now also U8.3
- net B: now also U8.4
- net DIR_Servo: now also U7.5
- net ENA_Servo: now also U7.4
- net GND: now also U7.1, U7.10, U7.12, U7.8, U8.2, U8.6, U8.7
- net I2C1_SCL: now also U8.9
- net I2C1_SDA: now also U8.10
- net PWM2_OUT: now also U7.11
- net PWM_Heater: now also U7.9
- net PWM_Servo: now also U7.6
- net T+: now also U8.5
- net ULN_EXTRA_1: now also U7.2
- net ULN_EXTRA_2: now also U7.3

Commit message: finish v1.0
Parts:
- removed D10: FR107, Diode_SMD:D_SMA, symbol Device:D
- added D10: SS54, Diode_SMD:D_SMA, symbol Diode:1N5711
Connections:
- net LCD_MOSI is gone; now on net LCD_DATA: U2.16 (B2)
- net +24V Servo: now also D10.1 (K); no longer D17.1 (K), D8.1 (K), F1.1, U8.1
- net BT1: now also C37.1, R32.1, SW2.2
- net BT2: now also C38.1, R33.1, SW3.2
- net CTR_DIR: now also U6.4 (I4); no longer U6.2 (I2)
- net DIR_Servo: now also U6.15 (O4); no longer U6.17 (O2)
- net EXTRA_1: now also U6.2 (I2); no longer U6.5 (I5)
- net EXTRA_2: now also U6.1 (I1); no longer U6.6 (I6)
- net GND: now also U6.6 (I6)
- net PWM_2: now also U6.5 (I5); no longer U6.1 (I1)
- net PWM_Servo: now also D10.2 (A)
- net ULN_EXTRA_1: now also U6.17 (O2), U7.3; no longer U6.14 (O5), U7.2
- net ULN_EXTRA_2: now also U6.18 (O1), U7.2; no longer U6.13 (O6), U7.3
- net ULN_PWM_2: now also U6.14 (O5); no longer U6.18 (O1)
- new net VIN: D17.1 (K), D8.1 (K), F1.1, U8.1
- no-connect marks 17 -> 18
